Commit message: Feature : skid robot done

File: gcamp_gazebo/urdf/skidbot.xacro (robot description, xacro)
@@ -1,6 +1,6 @@
 <?xml version='1.0'?>
 <robot name="bocbot" xmlns:xacro="http://www.ros.org/wiki/xacro">
+  <link name="robot_footprint"></link>
   <xacro:include filename="$(find gcamp_gazebo)/urdf/skidbot.gazebo" />
-  <link name="robot_footprint"></link>
   <joint name="robot_footprint_joint" type="fixed">
     <origin xyz="0 0 0" rpy="0 0 0" />
@@ -30,5 +30,5 @@
   <link name="front_left_wheel">
     <inertial>
-      <mass value="5.0" />
+      <mass value="8.0" />
       <origin xyz="0.0 0 0" rpy=" 0 1.5707 1.5707" />
       <inertia ixx="0.1" ixy="0" ixz="0" iyy="0.1" iyz="0" izz="0.1" />
@@ -49,5 +49,5 @@
   <link name="back_left_wheel">
     <inertial>
-      <mass value="5.0" />
+      <mass value="8.0" />
       <origin xyz="0.0 0 0" rpy=" 0 1.5707 1.5707" />
       <inertia ixx="0.1" ixy="0" ixz="0" iyy="0.1" iyz="0" izz="0.1" />
@@ -68,5 +68,5 @@
   <link name="front_right_wheel">
     <inertial>
-      <mass value="5.0" />
+      <mass value="8.0" />
       <origin xyz="0.0 0 0" rpy=" 0 1.5707 1.5707" />
       <inertia ixx="0.1" ixy="0" ixz="0" iyy="0.1" iyz="0" izz="0.1" />
@@ -87,5 +87,5 @@
   <link name="back_right_wheel">
     <inertial>
-      <mass value="5.0" />
+      <mass value="8.0" />
       <origin xyz="0.0 0 0" rpy=" 0 1.5707 1.5707" />
       <inertia ixx="0.1" ixy="0" ixz="0" iyy="0.1" iyz="0" izz="0.1" />
@@ -149,5 +149,5 @@
     <axis xyz="0 1 0" rpy="0 0 0" />
     <limit effort="10000" velocity="1000" />
-    <dynamics damping="1.0" friction="1.0" />
+    <dynamics damping="1.0" friction="5.0" />
   </joint>
   <joint type="continuous" name="front_right_wheel_joint">
@@ -157,5 +157,5 @@
     <axis xyz="0 1 0" rpy="0 0 0" />
     <limit effort="10000" velocity="1000" />
-    <dynamics damping="1.0" friction="1.0" />
+    <dynamics damping="1.0" friction="5.0" />
   </joint>
   <joint type="continuous" name="back_left_wheel_joint">
@@ -165,5 +165,5 @@
     <axis xyz="0 1 0" rpy="0 0 0" />
     <limit effort="10000" velocity="1000" />
-    <dynamics damping="1.0" friction="1.0" />
+    <dynamics damping="1.0" friction="5.0" />
   </joint>
   <joint type="continuous" name="back_right_wheel_joint">
@@ -173,5 +173,5 @@
     <axis xyz="0 1 0" rpy="0 0 0" />
     <limit effort="10000" velocity="1000" />
-    <dynamics damping="1.0" friction="1.0" />
+    <dynamics damping="1.0" friction="5.0" />
   </joint>
   <joint type="fixed" name="camera_joint">

Commit message: Update : various robot model added done

File: gcamp_gazebo/urdf/skidbot.xacro (robot description, xacro)
@@ -144,5 +144,5 @@
   </link>
   <joint type="continuous" name="front_left_wheel_joint">
-    <origin xyz="0.12 0.15 0" rpy="0 0 0" />
+    <origin xyz="0.13 0.15 0" rpy="0 0 0" />
     <child link="front_left_wheel" />
     <parent link="chassis" />
@@ -152,5 +152,5 @@
   </joint>
   <joint type="continuous" name="front_right_wheel_joint">
-    <origin xyz="0.12 -0.15 0" rpy="0 0 0" />
+    <origin xyz="0.13 -0.15 0" rpy="0 0 0" />
     <child link="front_right_wheel" />
     <parent link="chassis" />
@@ -160,5 +160,5 @@
   </joint>
   <joint type="continuous" name="back_left_wheel_joint">
-    <origin xyz="-0.12 0.15 0" rpy="0 0 0" />
+    <origin xyz="-0.13 0.15 0" rpy="0 0 0" />
     <child link="back_left_wheel" />
     <parent link="chassis" />
@@ -168,5 +168,5 @@
   </joint>
   <joint type="continuous" name="back_right_wheel_joint">
-    <origin xyz="-0.12 -0.15 0" rpy="0 0 0" />
+    <origin xyz="-0.13 -0.15 0" rpy="0 0 0" />
     <child link="back_right_wheel" />
     <parent link="chassis" />

File: gcamp_gazebo/urdf/trackbot.xacro (robot description, xacro)
@@ -11,10 +11,10 @@
     <pose frame=''>0 0 0 0 0 0</pose>
     <inertial>
-      <origin xyz="-0.122 0 0.118" rpy="1.5708 -0 0" />
+      <origin xyz="0.0 0 0.118" rpy="1.5708 -0 0" />
       <mass value="13.14" />
       <inertia ixx="0.10019" ixy="0.0" ixz="0.0" iyy="0.345043" iyz="0.0" izz="0.302044" />
     </inertial>
     <collision name='base_link_collision'>
-      <origin xyz="-0.122 0 0.118" rpy="0 -0 0" />
+      <origin xyz="0.0 0 0.118" rpy="0 -0 0" />
       <geometry>
         <box size="0.50017 0.24093 0.139" />
@@ -22,5 +22,5 @@
     </collision>
     <visual name='base_link_visual'>
-      <origin xyz="-0.122 0 0.118" rpy="0 -0 0" />
+      <origin xyz="0.0 0 0.118" rpy="0 -0 0" />
       <geometry>
         <box size="0.50017 0.24093 0.139" />
@@ -37,5 +37,5 @@
       <origin xyz="0.0 0 0" rpy=" 0 1.5707 1.5707" />
       <geometry>
-        <cylinder length="0.05" radius="0.1" />
+        <cylinder length="0.09728" radius="0.12" />
       </geometry>
     </visual>
@@ -43,5 +43,5 @@
       <origin xyz="0.0 0 0" rpy=" 0 1.5707 1.5707" />
       <geometry>
-        <cylinder length="0.05" radius="0.1" />
+        <cylinder length="0.09728" radius="0.12" />
       </geometry>
     </collision>
@@ -56,5 +56,5 @@
       <origin xyz="0.0 0 0" rpy=" 0 1.5707 1.5707" />
       <geometry>
-        <cylinder length="0.05" radius="0.1" />
+        <cylinder length="0.09728" radius="0.12" />
       </geometry>
     </visual>
@@ -62,5 +62,5 @@
       <origin xyz="0.0 0 0" rpy=" 0 1.5707 1.5707" />
       <geometry>
-        <cylinder length="0.05" radius="0.1" />
+        <cylinder length="0.09728" radius="0.12" />
       </geometry>
     </collision>
@@ -75,5 +75,5 @@
       <origin xyz="0.0 0 0" rpy=" 0 1.5707 1.5707" />
       <geometry>
-        <cylinder length="0.05" radius="0.1" />
+        <cylinder length="0.09728" radius="0.12" />
       </geometry>
     </visual>
@@ -81,5 +81,5 @@
       <origin xyz="0.0 0 0" rpy=" 0 1.5707 1.5707" />
       <geometry>
-        <cylinder length="0.05" radius="0.1" />
+        <cylinder length="0.09728" radius="0.12" />
       </geometry>
     </collision>
@@ -94,5 +94,5 @@
       <origin xyz="0.0 0 0" rpy=" 0 1.5707 1.5707" />
       <geometry>
-        <cylinder length="0.05" radius="0.1" />
+        <cylinder length="0.09728" radius="0.12" />
       </geometry>
     </visual>
@@ -100,10 +100,10 @@
       <origin xyz="0.0 0 0" rpy=" 0 1.5707 1.5707" />
       <geometry>
-        <cylinder length="0.05" radius="0.1" />
+        <cylinder length="0.09728" radius="0.12" />
       </geometry>
     </collision>
   </link>
   <joint type="continuous" name="front_left_wheel_joint">
-    <origin xyz="0.12 0.15 0" rpy="0 0 0" />
+    <origin xyz="0.15 0.1985 0.01855" rpy="0 0 0" />
     <child link="front_left_wheel" />
     <parent link="base_link" />
@@ -113,5 +113,5 @@
   </joint>
   <joint type="continuous" name="front_right_wheel_joint">
-    <origin xyz="0.12 -0.15 0" rpy="0 0 0" />
+    <origin xyz="0.15 -0.1985 0.01855" rpy="0 0 0" />
     <child link="front_right_wheel" />
     <parent link="base_link" />
@@ -121,5 +121,5 @@
   </joint>
   <joint type="continuous" name="back_left_wheel_joint">
-    <origin xyz="-0.12 0.15 0" rpy="0 0 0" />
+    <origin xyz="-0.15 0.1985 0.01855" rpy="0 0 0" />
     <child link="back_left_wheel" />
     <parent link="base_link" />
@@ -129,5 +129,5 @@
   </joint>
   <joint type="continuous" name="back_right_wheel_joint">
-    <origin xyz="-0.12 -0.15 0" rpy="0 0 0" />
+    <origin xyz="-0.15 -0.1985 0.01855" rpy="0 0 0" />
     <child link="back_right_wheel" />
     <parent link="base_link" />
